File: hvpsu.kicad_pcb (KiCad board)
At the start: 2 copper layers, 0 parts

Commit message: autospread all components on the pcb
Parts:
- added C1: 680uF, Capacitors_ThroughHole:C_Radial_D35_L51_P10, F.Cu at (154.1, 135.0)
- added C2: 680uF, Capacitors_ThroughHole:C_Radial_D35_L51_P10, F.Cu at (118.1, 135.0)
- added D1: KBU10M, bridges:KBU10M_Bridge_Rectifier_1000V, F.Cu at (189.9, 125.9)
- added F1: FUSE, Fuse_Holders_and_Fuses:Fuseholder5x20_horiz_open_universal_Type-III, F.Cu at (200.4, 76.4)
- added P1: CONN_01X02, Terminal_Blocks:TerminalBlock_WAGO-236_2Stift_RM5mm_2pol, F.Cu at (193.7, 93.8)
- added P2: CONN_01X02, Terminal_Blocks:TerminalBlock_WAGO-236_2Stift_RM5mm_2pol, F.Cu at (219.9, 80.3)
- added R1: 1k, Resistors_ThroughHole:Resistor_Ceramic_Horizontal_L65mm-W16mm-H15mm-p80mm, F.Cu at (146.2, 81.5)
- added R10: 1k, Resistors_ThroughHole:Resistor_Ceramic_Horizontal_L65mm-W16mm-H15mm-p80mm, F.Cu at (146.2, 59.1)
- added R11: 1k, Resistors_ThroughHole:Resistor_Ceramic_Horizontal_L65mm-W16mm-H15mm-p80mm, F.Cu at (64.0, 81.5)
- added R12: 1k, Resistors_ThroughHole:Resistor_Ceramic_Horizontal_L65mm-W16mm-H15mm-p80mm, F.Cu at (146.2, 36.7)
- added R13: 1k, Resistors_ThroughHole:Resistor_Ceramic_Horizontal_L65mm-W16mm-H15mm-p80mm, F.Cu at (64.0, 59.1)
- added R2: 1k, Resistors_ThroughHole:Resistor_Ceramic_Horizontal_L65mm-W16mm-H15mm-p80mm, F.Cu at (146.2, 103.9)
- added R3: 1k, Resistors_ThroughHole:Resistor_Ceramic_Horizontal_L65mm-W16mm-H15mm-p80mm, F.Cu at (228.4, 59.1)
- added R4: 1k, Resistors_ThroughHole:Resistor_Ceramic_Horizontal_L65mm-W16mm-H15mm-p80mm, F.Cu at (64.0, 36.7)
- added R5: 1k, Resistors_ThroughHole:Resistor_Ceramic_Horizontal_L65mm-W16mm-H15mm-p80mm, F.Cu at (64.0, 148.8)
- added R6: 0R, Resistors_ThroughHole:Resistor_Ceramic_Horizontal_L65mm-W16mm-H15mm-p80mm, F.Cu at (228.4, 36.7)
- added R7: 0R, Resistors_ThroughHole:Resistor_Ceramic_Horizontal_L65mm-W16mm-H15mm-p80mm, F.Cu at (64.0, 126.4)
- added R9: 1k, Resistors_ThroughHole:Resistor_Ceramic_Horizontal_L65mm-W16mm-H15mm-p80mm, F.Cu at (64.0, 103.9)
- added SW1: Switch_DPST, switches:DPST_Rocker_Switch_Chily_3024_Angled, F.Cu at (233.6, 79.8)
